Commit message: dragging_RL_06022020

File: ROBOTIS-THORMANG-Common/thormang3_description/urdf/thormang3.structure.arm.xacro (robot description, xacro)
@@ -240,4 +240,9 @@
 	<!-- left arm gripper link -->
         <link name="l_arm_grip_link">
+		  <collision>
+      	    <geometry>
+              <mesh filename="package://thormang3_description/meshes/robotis_l_arm_grip_link.stl" scale="0.001 0.001 0.001"/>
+      	    </geometry>
+    	  </collision>
    	  <visual>
       	    <origin xyz="0 0 0" rpy="0 0 0"/>
@@ -266,4 +271,9 @@
 	<!-- left arm gripper 1 link -->
         <link name="l_arm_grip_1_link">
+		  <collision>
+      	    <geometry>
+              <mesh filename="package://thormang3_description/meshes/robotis_l_arm_grip_1_link.stl" scale="0.001 0.001 0.001"/>
+      	    </geometry>
+    	  </collision>
    	  <visual>
       	    <origin xyz="0 0 0" rpy="0 0 0"/>
@@ -539,4 +549,9 @@
 	<!-- right arm gripper link -->
         <link name="r_arm_grip_link">
+    	  <collision>
+      	    <geometry>
+			   <mesh filename="package://thormang3_description/meshes/robotis_r_arm_grip_1_link.stl" scale="0.001 0.001 0.001"/>
+      	    </geometry>
+    	  </collision>
    	  <visual>
       	    <origin xyz="0 0 0" rpy="0 0 0"/>
@@ -565,4 +580,9 @@
 	<!-- right arm gripper link -->
         <link name="r_arm_grip_1_link">
+		  <collision>
+      	    <geometry>
+              <mesh filename="package://thormang3_description/meshes/robotis_r_arm_grip_link.stl" scale="0.001 0.001 0.001"/>
+      	    </geometry>
+    	  </collision>
    	  <visual>
       	    <origin xyz="0 0 0" rpy="0 0 0"/>
